File: pcb/updi_ki.kicad_pcb (KiCad board)
At the start: 2 copper layers, 56.5 x 21.6 mm, 36 parts, among them J2 UPDI-IN, J3 UPDI_IN6, J4 HVUPDI_OUT6, J5 HVUPDI-OUT, SW1 SN74LVC1G3157DBVR, SW2 ISL43210IHZ-T, SW3 PTS810SJG250SMTRLFS, U1 ATtiny202-SS, U2 NCP1406SNT1G, U3 MIC2091-1YM5-TR

Commit message: Condense layout
Signed-off-by: Michael Darr <michael.e.darr@gmail.com>
Parts:
- removed FID1, FID2, FID3, FID4: Fiducial, Fiducial:Fiducial_1mm_Mask2mm
- removed J2: UPDI-IN, Connector_PinHeader_2.54mm:PinHeader_1x03_P2.54mm_Horizontal
- removed J5: HVUPDI-OUT, Connector_PinSocket_2.54mm:PinSocket_1x03_P2.54mm_Horizontal
- added JP1: SolderJumper_2_Bridged, Jumper:SolderJumper-2_P1.3mm_Bridged_RoundedPad1.0x1.5mm, F.Cu at (117.1, 50.0)
- moved C3 82.2 mm to (127.6, 66.1), turned to -90 degrees
- moved C8 79.5 mm to (125.5, 66.1), turned to -90 degrees
- moved C1 78.4 mm to (121.0, 58.5)
- moved U1 78.0 mm to (123.2, 54.5)
- moved F1 77.0 mm to (105.1, 50.0), turned to 90 degrees
- moved R4 76.7 mm to (123.5, 66.1), turned to -90 degrees
- moved L1 75.6 mm to (108.8, 50.3)
- moved U2 74.9 mm to (107.9, 54.1)
- moved D2 74.8 mm to (113.2, 49.5)
- moved C4 74.8 mm to (113.2, 57.2)
- moved C6 74.8 mm to (113.2, 59.7)
- moved C7 74.8 mm to (113.2, 62.3)
- moved R10 74.8 mm to (108.6, 59.7)
- moved R12 74.8 mm to (113.2, 64.8)
- moved R5 74.8 mm to (113.2, 54.5)
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Connections:
- net /UPDI-HOST renamed UPDI-HOST
- J3 pad 3: /PROG -> unconnected-(J3-Pin_3-Pad3)
- J3 pad 4: (no net) -> unconnected-(J3-Pin_4-Pad4)
- J3 pad 5: (no net) -> unconnected-(J3-Pin_5-Pad5)
- J4 pad 3: VTG -> unconnected-(J4-Pin_3-Pad3)
- J4 pad 4: (no net) -> unconnected-(J4-Pin_4-Pad4)
- J4 pad 5: (no net) -> unconnected-(J4-Pin_5-Pad5)
- U1 pad 6: /PROG -> Net-(JP1-A)
- U3 pad 4: (no net) -> unconnected-(U3-FAULT/-Pad4)
Routing:
- net /HV-EN: track 83.9 -> 34.9 mm, vias 2 -> 0
- net VTG: track 89.9 -> 46.7 mm, vias 2 -> 0
- net /HVUPDI-TARGET: track 53.3 -> 12.6 mm, vias 0 -> 2
- net /PROG: track 36.1 -> 0.00 mm, vias 1 -> 0
- net /UPDI-EN: track 47.2 -> 19.4 mm, vias 2 -> 0
- net UPDI-HOST: track 43.1 -> 24.7 mm
- net /UPDI-SENSE: track 31.3 -> 45.3 mm
- net GND: track 58.7 -> 48.7 mm, vias 8 -> 9
- net /PWR-SW-EN: track 11.3 -> 20.1 mm
- net VF: track 60.1 -> 51.4 mm, vias 2 -> 0
- net /UPDI-KEY: track 10.2 -> 2.98 mm
- net VTG-PC: track 40.9 -> 34.4 mm
- net Net-(VTG1-A): track 7.57 -> 1.99 mm
- net Net-(JP1-A): track 0.00 -> 5.37 mm
- net /12V: track 34.7 -> 29.8 mm, vias 2 -> 0
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Other:
- board size 56.5 x 21.6 mm -> 30.3 x 21.1 mm
- rule pad_to_mask_clearance: 0.051 -> 0
- board text added: "HOST"
- board text added: "TARGET"
- board text added: "UPDI-KI"
- board text added: "rev 0.1.0"
- board text added: "Ü"
- board text added: "╔═══════╗ ║ ║ ╚═══════╝"
- board text added: "✂"
- board text removed: "4E564D50726F6720"
- board text removed: "DAT"
- board text removed: "GND"
- board text removed: "HV-UPDI-TARGET"
- board text removed: "HVUPDI"
- board text removed: "PROG"
- board text removed: "UPDI"
- board text removed: "UPDI-HOST"
- board text removed: "Updi-Key"
- board text removed: "VTG-PC"
- board text removed: "github.com/MichaelDarr/updi-ki"
- board text removed: "v1.0"
