File: pcb/updi_ki.kicad_sch (KiCad schematic)
At the start: 36 parts, among them J2 UPDI-IN, J3 UPDI_IN6, J4 HVUPDI_OUT6, J5 HVUPDI-OUT, SW1 SN74LVC1G3157DBVR, SW2 ISL43210IHZ-T, SW3 PTS810SJG250SMTRLFS, U1 ATtiny202-SS, U2 NCP1406SNT1G, U3 MIC2091-1YM5-TR

Commit message: Condense layout
Signed-off-by: Michael Darr <michael.e.darr@gmail.com>
Parts:
- removed FID1, FID2, FID3, FID4: Fiducial, Fiducial:Fiducial_1mm_Mask2mm, symbol Mechanical:Fiducial
- removed J2: UPDI-IN, Connector_PinHeader_2.54mm:PinHeader_1x03_P2.54mm_Horizontal, symbol Connector_Generic:Conn_01x03
- removed J5: HVUPDI-OUT, Connector_PinSocket_2.54mm:PinSocket_1x03_P2.54mm_Horizontal, symbol Connector_Generic:Conn_01x03
- added JP1: SolderJumper_2_Bridged, Jumper:SolderJumper-2_P1.3mm_Bridged_RoundedPad1.0x1.5mm, symbol Jumper:SolderJumper_2_Bridged
Connections:
- net UPDI-HOST: now also JP1.2 (B)
- net VTG: no longer J4.3 (Pin_3)
- net PROG: no longer names the net of U1.6 (~{RESET}/PA0)
- net PROG: now also JP1.1 (A); no longer J3.3 (Pin_3)
- no-connect marks 5 -> 7
Other:
- moved on the sheet: C2, C4, C6, C7, D2, HV1, J3, J4, L1, R10, R11, R12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
